File: PCB/pinky.kicad_sch (KiCad schematic)
At the start: 47 parts, among them SW1 SW_SPDT_321, SW10 MX_SW_HS, SW11 MX_SW_HS, SW12 MX_SW_HS, SW13 MX_SW_HS, SW14 MX_SW_HS, SW15 MX_SW_HS, SW16 MX_SW_HS, SW17 MX_SW_HS, SW18 MX_SW_HS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

Commit message: Rudimentary symbols clean up
Parts:
- JP2: symbol device_jumper_no_small:Device_Jumper_NO_Small -> Pinky:Device_Jumper_NO_Small
Changed lines of the file:
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@@
 	)
 	(symbol
-		(lib_id "device_jumper_no_small:Device_Jumper_NO_Small")
+		(lib_id "Pinky:Device_Jumper_NO_Small")
 		(at 45.72 118.11 0)
 		(unit 1)
