File: PCB/pinky.kicad_sch (KiCad schematic)
At the start: 47 parts, among them SW1 SW_SPDT_321, SW10 MX_SW_HS, SW11 MX_SW_HS, SW12 MX_SW_HS, SW13 MX_SW_HS, SW14 MX_SW_HS, SW15 MX_SW_HS, SW16 MX_SW_HS, SW17 MX_SW_HS, SW18 MX_SW_HS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

Commit message: Symbols rename and proper footprints assignment
Parts:
- JP1, JP2, JP3, JP4: value Device_Jumper_NO_Small -> Jumper; symbol Pinky:Device_Jumper_NO_Small -> Pinky:Jumper
- SW10, SW11, SW12, SW13, SW14, SW15, SW16, SW17, SW18, SW2, SW3, SW4, SW5, SW6, SW7, SW8, SW9: value MX_SW_HS -> Switch; symbol Pinky:MX_SW_HS -> Pinky:Switch
- U1: symbol Pinky:nice_nano -> Pinky:Nice!nano

Commit message: Footprint rename
Parts:
- SW10, SW11, SW12, SW13, SW14, SW15, SW16, SW17, SW18, SW2, SW3, SW4, SW5, SW6, SW7, SW8, SW9: footprint Pinky:Kailh_socket_PG1350_optional_reversible -> Pinky:SW_Kailh_Choc_PG1350
Changed lines of the file:
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@@
 			)
 		)
-		(property "Footprint" "Pinky:Kailh_socket_PG1350_optional_reversible"
+		(property "Footprint" "Pinky:SW_Kailh_Choc_PG1350"
 			(at 119.38 44.45 0)
 			(hide yes)
@@
 			)
 		)
-		(property "Footprint" "Pinky:Kailh_socket_PG1350_optional_reversible"
+		(property "Footprint" "Pinky:SW_Kailh_Choc_PG1350"
 			(at 140.97 26.67 0)
 			(hide yes)
@@
 			)
 		)
-		(property "Footprint" "Pinky:Kailh_socket_PG1350_optional_reversible"
+		(property "Footprint" "Pinky:SW_Kailh_Choc_PG1350"
 			(at 129.54 44.45 0)
 			(hide yes)
@@
 			)
 		)
-		(property "Footprint" "Pinky:Kailh_socket_PG1350_optional_reversible"
+		(property "Footprint" "Pinky:SW_Kailh_Choc_PG1350"
 			(at 119.38 26.67 0)
 			(hide yes)
@@
 			)
 		)
-		(property "Footprint" "Pinky:Kailh_socket_PG1350_optional_reversible"
+		(property "Footprint" "Pinky:SW_Kailh_Choc_PG1350"
 			(at 119.38 63.5 0)
 			(hide yes)
@@
 			)
 		)
-		(property "Footprint" "Pinky:Kailh_socket_PG1350_optional_reversible"
+		(property "Footprint" "Pinky:SW_Kailh_Choc_PG1350"
 			(at 96.52 81.28 0)
 			(hide yes)
@@
 			)
 		)
-		(property "Footprint" "Pinky:Kailh_socket_PG1350_optional_reversible"
+		(property "Footprint" "Pinky:SW_Kailh_Choc_PG1350"
 			(at 129.54 26.67 0)
 			(hide yes)
@@
 			)
 		)
-		(property "Footprint" "Pinky:Kailh_socket_PG1350_optional_reversible"
+		(property "Footprint" "Pinky:SW_Kailh_Choc_PG1350"
 			(at 107.95 63.5 0)
 			(hide yes)
@@
 			)
 		)
-		(property "Footprint" "Pinky:Kailh_socket_PG1350_optional_reversible"
+		(property "Footprint" "Pinky:SW_Kailh_Choc_PG1350"
 			(at 96.52 26.67 0)
 			(hide yes)
@@
 			)
 		)
-		(property "Footprint" "Pinky:Kailh_socket_PG1350_optional_reversible"
+		(property "Footprint" "Pinky:SW_Kailh_Choc_PG1350"
 			(at 140.97 44.45 0)
 			(hide yes)
@@
 			)
 		)
-		(property "Footprint" "Pinky:Kailh_socket_PG1350_optional_reversible"
+		(property "Footprint" "Pinky:SW_Kailh_Choc_PG1350"
 			(at 140.97 63.5 0)
 			(hide yes)
@@
 			)
 		)
-		(property "Footprint" "Pinky:Kailh_socket_PG1350_optional_reversible"
+		(property "Footprint" "Pinky:SW_Kailh_Choc_PG1350"
 			(at 96.52 63.5 0)
 			(hide yes)
@@
 			)
 		)
-		(property "Footprint" "Pinky:Kailh_socket_PG1350_optional_reversible"
+		(property "Footprint" "Pinky:SW_Kailh_Choc_PG1350"
 			(at 107.95 81.28 0)
 			(hide yes)
@@
 			)
 		)
-		(property "Footprint" "Pinky:Kailh_socket_PG1350_optional_reversible"
+		(property "Footprint" "Pinky:SW_Kailh_Choc_PG1350"
 			(at 107.95 44.45 0)
 			(hide yes)
@@
 			)
 		)
-		(property "Footprint" "Pinky:Kailh_socket_PG1350_optional_reversible"
+		(property "Footprint" "Pinky:SW_Kailh_Choc_PG1350"
 			(at 129.54 63.5 0)
 			(hide yes)
@@
 			)
 		)
-		(property "Footprint" "Pinky:Kailh_socket_PG1350_optional_reversible"
+		(property "Footprint" "Pinky:SW_Kailh_Choc_PG1350"
 			(at 107.95 26.67 0)
 			(hide yes)
@@
 			)
 		)
-		(property "Footprint" "Pinky:Kailh_socket_PG1350_optional_reversible"
+		(property "Footprint" "Pinky:SW_Kailh_Choc_PG1350"
 			(at 96.52 44.45 0)
 			(hide yes)

Commit message: Footprints assigned
Parts:
- D1, D10, D11, D12, D13, D14, D15, D16, D17, D2, D3, D4, D5, D6, D7, D8, D9: footprint (none) -> Pinky:Diode_SOD123
- H1, H2, H3, H4, H5: footprint (none) -> MountingHole:MountingHole_2.2mm_M2
Changed lines of the file:
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@@
 			)
 		)
-		(property "Footprint" ""
+		(property "Footprint" "MountingHole:MountingHole_2.2mm_M2"
 			(at 170.18 36.322 0)
 			(hide yes)
@@
 			)
 		)
-		(property "Footprint" ""
+		(property "Footprint" "Pinky:Diode_SOD123"
 			(at 110.49 55.88 90)
 			(hide yes)
@@
 			)
 		)
-		(property "Footprint" ""
+		(property "Footprint" "Pinky:Diode_SOD123"
 			(at 132.08 55.88 90)
 			(hide yes)
@@
 			)
 		)
-		(property "Footprint" ""
+		(property "Footprint" "Pinky:Diode_SOD123"
 			(at 99.06 38.1 90)
 			(hide yes)
@@
 			)
 		)
-		(property "Footprint" ""
+		(property "Footprint" "Pinky:Diode_SOD123"
 			(at 132.08 74.93 90)
 			(hide yes)
@@
 			)
 		)
-		(property "Footprint" ""
+		(property "Footprint" "Pinky:Diode_SOD123"
 			(at 110.49 74.93 90)
 			(hide yes)
@@
 			)
 		)
-		(property "Footprint" ""
+		(property "Footprint" "MountingHole:MountingHole_2.2mm_M2"
 			(at 170.18 29.972 0)
 			(hide yes)
@@
 			)
 		)
-		(property "Footprint" ""
+		(property "Footprint" "Pinky:Diode_SOD123"
 			(at 99.06 74.93 90)
 			(hide yes)
@@
 			)
 		)
-		(property "Footprint" ""
+		(property "Footprint" "MountingHole:MountingHole_2.2mm_M2"
 			(at 170.18 23.622 0)
 			(hide yes)
@@
 			)
 		)
-		(property "Footprint" ""
+		(property "Footprint" "Pinky:Diode_SOD123"
 			(at 110.49 38.1 90)
 			(hide yes)
@@
 			)
 		)
-		(property "Footprint" ""
+		(property "Footprint" "Pinky:Diode_SOD123"
 			(at 143.51 74.93 90)
 			(hide yes)
@@
 			)
 		)
-		(property "Footprint" ""
+		(property "Footprint" "Pinky:Diode_SOD123"
 			(at 110.49 92.71 90)
 			(hide yes)
@@
 			)
 		)
-		(property "Footprint" ""
+		(property "Footprint" "Pinky:Diode_SOD123"
 			(at 121.92 55.88 90)
 			(hide yes)
@@
 			)
 		)
-		(property "Footprint" ""
+		(property "Footprint" "MountingHole:MountingHole_2.2mm_M2"
 			(at 170.18 49.53 0)
 			(hide yes)
@@
 			)
 		)
-		(property "Footprint" ""
+		(property "Footprint" "Pinky:Diode_SOD123"
 			(at 99.06 55.88 90)
 			(hide yes)
@@
 			)
 		)
-		(property "Footprint" ""
+		(property "Footprint" "MountingHole:MountingHole_2.2mm_M2"
 			(at 170.18 42.926 0)
 			(hide yes)
@@
 			)
 		)
-		(property "Footprint" ""
+		(property "Footprint" "Pinky:Diode_SOD123"
 			(at 99.06 92.71 90)
 			(hide yes)
@@
 			)
 		)
-		(property "Footprint" ""
+		(property "Footprint" "Pinky:Diode_SOD123"
 			(at 132.08 38.1 90)
 			(hide yes)
@@
 			)
 		)
-		(property "Footprint" ""
+		(property "Footprint" "Pinky:Diode_SOD123"
 			(at 121.92 38.1 90)
 			(hide yes)
@@
 			)
 		)
-		(property "Footprint" ""
+		(property "Footprint" "Pinky:Diode_SOD123"
 			(at 121.92 74.93 90)
 			(hide yes)
@@
 			)
 		)
-		(property "Footprint" ""
+		(property "Footprint" "Pinky:Diode_SOD123"
 			(at 143.51 55.88 90)
 			(hide yes)
@@
 			)
 		)
-		(property "Footprint" ""
+		(property "Footprint" "Pinky:Diode_SOD123"
 			(at 143.51 38.1 90)
 			(hide yes)
