File: PCB/pinky.kicad_pcb (KiCad board)
At the start: 2 copper layers, 120.5 x 85.5 mm, 47 parts, among them SW1 SW_SPDT_321, SW10 Switch, SW11 Switch, SW12 Switch, SW13 Switch, SW14 Switch, SW15 Switch, SW16 Switch, SW17 Switch, SW18 Switch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

Commit message: PCB pulled updates
Parts:
- D1, D10, D11, D12, D13, D14, D15, D16, D17, D2, D3, D4, D5, D6, D7, D8, D9: value D_Small -> D; footprint Pinky:Diode_SOD123 -> Pinky:D_SOD123
- JP1, JP2, JP3, JP4: value Jumper -> SDA
- SW10, SW11, SW12, SW13, SW14, SW15, SW16, SW17, SW18, SW2, SW3, SW4, SW5, SW6, SW7, SW8, SW9: value Switch -> SW_Kailh_Choc_PG1350; footprint Pinky:SW_Kailh_Choc_PG1350 -> Pinky:Switch
